File: 1. PCB/GBC USB-C Charging Kit.brd (EAGLE design)
At the start: 21.5 x 32.9 mm, 31 parts, among them IC1 TP4056, IC2 8205A, IC3 DW01A, J1 USB-C, J2 GBC POWER JACK, J3 JST-SH-1MM, J4 GBC LED, J5 GBC LED-E

Commit message: Added “R” to any resistance with a value less than 1K
Parts:
- R5: value 100 -> 100R
- R7, R8, R9: value 330 -> 330R
Changed lines of the file:
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@@
 <layer number="20" name="Dimension" color="15" fill="1" visible="yes" active="yes"/>
 <layer number="21" name="tPlace" color="7" fill="1" visible="yes" active="yes"/>
-<layer number="22" name="bPlace" color="7" fill="1" visible="yes" active="yes"/>
+<layer number="22" name="bPlace" color="7" fill="1" visible="no" active="yes"/>
 <layer number="23" name="tOrigins" color="15" fill="1" visible="yes" active="yes"/>
-<layer number="24" name="bOrigins" color="15" fill="1" visible="yes" active="yes"/>
+<layer number="24" name="bOrigins" color="15" fill="1" visible="no" active="yes"/>
 <layer number="25" name="tNames" color="7" fill="1" visible="no" active="yes"/>
 <layer number="26" name="bNames" color="7" fill="1" visible="no" active="yes"/>
@@
 <attribute name="NAME" x="6.6" y="16.891" size="0.9144" layer="21" font="vector" ratio="12" align="center-left"/>
 </element>
-<element name="R7" library=",giltesa" package="R0402" value="330" x="19.939" y="12.744" smashed="yes" rot="R270">
+<element name="R7" library=",giltesa" package="R0402" value="330R" x="19.939" y="12.744" smashed="yes" rot="R270">
 <attribute name="NAME" x="19.304" y="14.728" size="0.9144" layer="21" font="vector" ratio="12" align="center-left"/>
 </element>
-<element name="R8" library=",giltesa" package="R0402" value="330" x="19.939" y="9.696" smashed="yes" rot="R270">
+<element name="R8" library=",giltesa" package="R0402" value="330R" x="19.939" y="9.696" smashed="yes" rot="R270">
 <attribute name="NAME" x="19.304" y="7.747" size="0.9144" layer="21" font="vector" ratio="12" align="center-left"/>
 </element>
@@
 <attribute name="NAME" x="10.16" y="5.842" size="0.9144" layer="21" font="vector" ratio="12" rot="R90" align="center-left"/>
 </element>
-<element name="R5" library=",giltesa" package="R0402" value="100" x="7.8573" y="19.939" smashed="yes" rot="R180">
+<element name="R5" library=",giltesa" package="R0402" value="100R" x="7.8573" y="19.939" smashed="yes" rot="R180">
 <attribute name="NAME" x="5.965" y="19.3167" size="0.9144" layer="21" font="vector" ratio="12" rot="R90" align="center-left"/>
 </element>
@@
 <element name="J2" library=",giltesa" package="GBC_POWER_JACK_2" value="GBC POWER JACK" x="3.524" y="-0.635" smashed="yes"/>
 <element name="JP1" library="SparkFun-Jumpers" package="SMT-JUMPER_3_NO_SILK" value="JUMPER" x="5.3975" y="9.841" smashed="yes"/>
-<element name="R9" library=",giltesa" package="R0402" value="330" x="18.383" y="-2.032" smashed="yes">
+<element name="R9" library=",giltesa" package="R0402" value="330R" x="18.383" y="-2.032" smashed="yes">
 <attribute name="NAME" x="20.2118" y="-2.921" size="0.9144" layer="21" font="vector" ratio="12" rot="SR270" align="center-left"/>
 </element>
