File: 1. PCB/GBC USB-C Charging Kit.sch (EAGLE design)
At the start: 31 parts, among them IC1 TP4056, IC2 8205A, IC3 DW01A, J1 USB-C, J2 GBC POWER JACK, J3 JST-SH-1MM, J4 GBC LED, J5 GBC LED-E

Commit message: Added “R” to any resistance with a value less than 1K
Parts:
- R5: value 100 -> 100R
- R7, R8, R9: value 330 -> 330R
Changed lines of the file:
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@@
 <setting verticaltext="up"/>
 </settings>
-<grid distance="100" unitdist="mil" unit="mil" style="lines" multiple="1" display="no" altdistance="0.01" altunitdist="inch" altunit="inch"/>
+<grid distance="0.1" unitdist="inch" unit="inch" style="lines" multiple="1" display="no" altdistance="0.01" altunitdist="inch" altunit="inch"/>
 <layers>
 <layer number="1" name="Top" color="4" fill="1" visible="no" active="no"/>
@@
 <part name="C2" library=",giltesa" deviceset="C0603" device="" value="100nF"/>
 <part name="IC2" library="SparkFun" deviceset="FS8205A" device="" value="8205A"/>
-<part name="R5" library=",giltesa" deviceset="R0402" device="" value="100"/>
+<part name="R5" library=",giltesa" deviceset="R0402" device="" value="100R"/>
 <part name="R6" library=",giltesa" deviceset="R0402" device="" value="1k"/>
-<part name="R7" library=",giltesa" deviceset="R0402" device="" value="330"/>
-<part name="R8" library=",giltesa" deviceset="R0402" device="" value="330"/>
+<part name="R7" library=",giltesa" deviceset="R0402" device="" value="330R"/>
+<part name="R8" library=",giltesa" deviceset="R0402" device="" value="330R"/>
 <part name="GND12" library="SparkFun" deviceset="GND" device=""/>
 <part name="GND-ISO3" library="SparkFun-PowerSymbols" deviceset="GND-ISO" device="" value="GND-BAT"/>
@@
 <part name="GND9" library="SparkFun" deviceset="GND" device=""/>
 <part name="JP1" library="SparkFun-Jumpers" deviceset="JUMPER-SMT_3_NO" device="_SILK" value="JUMPER"/>
-<part name="R9" library=",giltesa" deviceset="R0402" device="" value="330"/>
+<part name="R9" library=",giltesa" deviceset="R0402" device="" value="330R"/>
 <part name="J4" library=",giltesa" deviceset="1X03" device="2" value="GBC LED"/>
 <part name="J5" library=",giltesa" deviceset="GBC_LED" device="" value="GBC LED-E"/>
